Commit message: in work. not gazebo ready

File: lobster/urdf/lobster.urdf.xacro (robot description, xacro)
@@ -1,9 +1,10 @@
 <?xml version="1.0"?>
 <robot xmlns:xacro="http://www.ros.org/wiki/xacro" name="lobster">
-    <xacro:include filename="material.xacro" />
-    <xacro:include filename="lobster.xacro" />
-    <xacro:include filename="joints.xacro" />
+    <xacro:include filename="material2.xacro" />
+    <xacro:include filename="lobster_chassi.xacro"/>
+    <xacro:include filename="lobster_body.xacro"/>
+<!--
     <xacro:include filename="display.xacro" />
-    <xacro:include filename="camera.xacro" />
+    <xacro:include filename="camera.xacro" /> -->
     <xacro:include filename="lidar.xacro" />
  <!--    <xacro:include filename="gazebo.xacro"/>  -->

File: lobster/urdf/lobster_body.xacro (robot description, xacro)
@@ -6,5 +6,5 @@
             <origin xyz="0.0 0.0 0.0" rpy="0.0 0.0 0.0"/>
             <geometry>
-                <mesh filename="package://test_pkg/meshes/meshes_Homebot/body/LowerCover-Part1.stl" scale="${scale}"/>
+                <mesh filename="package://lobster/meshes/body/LowerCover-Part1.stl" scale="${scale}"/>
             </geometry>
             <material name="red"/>
@@ -20,5 +20,5 @@
             <origin xyz="0.0 0.0 0.0" rpy="0.0 0.0 0.0"/>
             <geometry>
-                <mesh filename="package://test_pkg/meshes/meshes_Homebot/body/LowerCover-Part2.stl" scale="${scale}"/>
+                <mesh filename="package://lobster/meshes/body/LowerCover-Part2.stl" scale="${scale}"/>
             </geometry>
             <material name="red"/>
@@ -34,5 +34,5 @@
             <origin xyz="0.0 0.0 0.0" rpy="0.0 0.0 0.0"/>
             <geometry>
-                <mesh filename="package://test_pkg/meshes/meshes_Homebot/body/LowerCover-Part3.stl" scale="${scale}"/>
+                <mesh filename="package://lobster/meshes/body/LowerCover-Part3.stl" scale="${scale}"/>
             </geometry>
             <material name="red"/>
@@ -48,5 +48,5 @@
             <origin xyz="0.0 0.0 0.0" rpy="0.0 0.0 0.0"/>
             <geometry>
-                <mesh filename="package://test_pkg/meshes/meshes_Homebot/body/LowerCover-Part4.stl" scale="${scale}"/>
+                <mesh filename="package://lobster/meshes/body/LowerCover-Part4.stl" scale="${scale}"/>
             </geometry>
             <material name="red"/>
@@ -63,5 +63,5 @@
             <geometry>
                 <mesh
-                    filename="package://test_pkg/meshes/meshes_Homebot/body/UpperCover-Face-Part1.stl"
+                    filename="package://lobster/meshes/body/UpperCover-Face-Part1.stl"
                     scale="${scale}" />
             </geometry>
@@ -79,5 +79,5 @@
             <origin xyz="0.0 0.0 0.0" rpy="0.0 0.0 0.0"/>
             <geometry>
-                <mesh filename="package://test_pkg/meshes/meshes_Homebot/body/UpperCover-Part2.stl" scale="${scale}"/>
+                <mesh filename="package://lobster/meshes/body/UpperCover-Part2.stl" scale="${scale}"/>
             </geometry>
             <material name="red"/>
@@ -93,5 +93,5 @@
             <origin xyz="0.0 0.0 0.0" rpy="0.0 0.0 0.0"/>
             <geometry>
-                <mesh filename="package://test_pkg/meshes/meshes_Homebot/body/Upper_Cover-With_Servo-Part3.stl" scale="${scale}"/>
+                <mesh filename="package://lobster/meshes/body/Upper_Cover-With_Servo-Part3.stl" scale="${scale}"/>
             </geometry>
             <material name="red"/>
@@ -107,5 +107,5 @@
             <origin xyz="0.0 0.0 0.0" rpy="0.0 0.0 0.0"/>
             <geometry>
-                <mesh filename="package://test_pkg/meshes/meshes_Homebot/body/Upper_Cover-With_Servo-Part4.stl" scale="${scale}"/>
+                <mesh filename="package://lobster/meshes/body/Upper_Cover-With_Servo-Part4.stl" scale="${scale}"/>
             </geometry>
             <material name="red"/>
@@ -122,5 +122,5 @@
             <geometry>
                 <mesh
-                    filename="package://test_pkg/meshes/meshes_Homebot/body/LidarTopPlate.stl"
+                    filename="package://lobster/meshes/body/LidarTopPlate.stl"
                     scale="${scale}" />
             </geometry>

File: lobster/urdf/lobster_chassi.xacro (robot description, xacro)
@@ -7,5 +7,5 @@
             <origin xyz="0.0 0.0 0.0" rpy="0.0 0.0 ${-PI/2}"/>
             <geometry>
-                <mesh filename="package://test_pkg/meshes/meshes_Homebot/body/BasePlateHorizontal.stl" scale="${scale}"/>
+                <mesh filename="package://lobster/meshes/body/BasePlateHorizontal.stl" scale="${scale}"/>
             </geometry>
             <material name="blue"/>
@@ -21,5 +21,5 @@
             <origin xyz="0.0 0.0 0.0" rpy="0.0 0.0 0.0"/>
             <geometry>
-                <mesh filename="package://test_pkg/meshes/meshes_Homebot/body/wheel.dae" scale="0.5 0.5 0.5"/>
+                <mesh filename="package://lobster/meshes/body/wheel.dae" scale="0.5 0.5 0.5"/>
             </geometry>
         </visual>
@@ -35,13 +35,27 @@
             <origin xyz="0.0 0.0 0.0" rpy="0.0 0.0 ${PI}"/>
             <geometry>
-                <mesh filename="package://test_pkg/meshes/meshes_Homebot/body/wheel.dae" scale="0.5 0.5 0.5"/>
+                <mesh filename="package://lobster/meshes/body/wheel.dae" scale="0.5 0.5 0.5"/>
             </geometry>
         </visual>
     </link>
-    <joint name="right_wheel_joint" type="continuous">
+    <joint name="joint_1" type="continuous">
         <parent link="base_link"/>
         <child link="right_wheel"/>
         <axis xyz="0 1 0"/>
         <origin xyz="0 -0.12 0.02" rpy="0 0 0"/>
+    </joint>
+    <link name="left_wheel">
+        <visual>
+            <origin xyz="0.0 0.0 0.0" rpy="0.0 0.0 0.0"/>
+            <geometry>
+                <mesh filename="package://lobster/meshes/body/wheel.dae" scale="0.5 0.5 0.5"/>
+            </geometry>
+        </visual>
+    </link>
+    <joint name="joint_2" type="continuous">
+        <parent link="base_link"/>
+        <child link="left_wheel"/>
+        <axis xyz="0 1 0"/>
+        <origin xyz="0 0.12 0.02" rpy="0 0 0"/>
     </joint>
     <link name="caster_wheel_front">

File: lobster/urdf/rover.urdf.xacro (robot description, xacro)
@@ -2,5 +2,5 @@
 <robot xmlns:xacro="http://www.ros.org/wiki/xacro" name="rover">
     <xacro:include filename="material.xacro"/>
-    <xacro:include filename="rover_chassi.xacro"/>
-    <xacro:include filename="rover_body_n.xacro"/>
+    <xacro:include filename="lobster_chassi.xacro"/>
+    <xacro:include filename="lobster_body.xacro"/>
 </robot>

Commit message: in work see homer

File: lobster/urdf/lobster.urdf.xacro (robot description, xacro)
@@ -1,5 +1,5 @@
 <?xml version="1.0"?>
 <robot xmlns:xacro="http://www.ros.org/wiki/xacro" name="lobster">
-    <xacro:include filename="material2.xacro" />
+    <xacro:include filename="material.xacro" />
     <xacro:include filename="lobster_chassi.xacro"/>
     <xacro:include filename="lobster_body.xacro"/>

File: lobster/urdf/lobster_body.xacro (robot description, xacro)
@@ -4,57 +4,85 @@
     <link name="body_1">
         <visual>
-            <origin xyz="0.0 0.0 0.0" rpy="0.0 0.0 0.0"/>
-            <geometry>
-                <mesh filename="package://lobster/meshes/body/LowerCover-Part1.stl" scale="${scale}"/>
-            </geometry>
-            <material name="red"/>
-        </visual>
+            <origin xyz="0.0 0.0 0.0" rpy="0.0 0.0 0.0" />
+            <geometry>
+                <mesh filename="package://lobster/meshes/body/LowerCover-Part1.stl" scale="${scale}" />
+            </geometry>
+            <material name="red" />
+        </visual>
+        <collision>
+            <origin xyz="0.0 0.0 0.0" rpy="0.0 0.0 0.0" />
+            <geometry>
+                <mesh filename="package://lobster/meshes/body/LowerCover-Part1.stl" scale="${scale}" />
+            </geometry>
+        </collision>
+        <xacro:default_inertial mass="1" />
     </link>
     <joint name="lower_body_1" type="fixed">
-        <parent link="base_link"/>
-        <child link="body_1"/>
-        <origin xyz="-0.043 0.046 0.0" rpy="0.0 0.0 ${PI/2}"/>
+        <parent link="base_link" />
+        <child link="body_1" />
+        <origin xyz="-0.043 0.046 0.0" rpy="0.0 0.0 ${PI/2}" />
     </joint>
     <link name="body_2">
         <visual>
-            <origin xyz="0.0 0.0 0.0" rpy="0.0 0.0 0.0"/>
-            <geometry>
-                <mesh filename="package://lobster/meshes/body/LowerCover-Part2.stl" scale="${scale}"/>
-            </geometry>
-            <material name="red"/>
-        </visual>
+            <origin xyz="0.0 0.0 0.0" rpy="0.0 0.0 0.0" />
+            <geometry>
+                <mesh filename="package://lobster/meshes/body/LowerCover-Part2.stl" scale="${scale}" />
+            </geometry>
+            <material name="red" />
+        </visual>
+        <collision>
+            <origin xyz="0.0 0.0 0.0" rpy="0.0 0.0 0.0" />
+            <geometry>
+                <mesh filename="package://lobster/meshes/body/LowerCover-Part2.stl" scale="${scale}" />
+            </geometry>
+        </collision>
+        <xacro:default_inertial mass="1" />
     </link>
     <joint name="lower_body_2" type="fixed">
-        <parent link="base_link"/>
-        <child link="body_2"/>
-        <origin xyz="-0.043 0.046 0" rpy="0.0 0.0 ${PI/2}"/>
+        <parent link="base_link" />
+        <child link="body_2" />
+        <origin xyz="-0.043 0.046 0" rpy="0.0 0.0 ${PI/2}" />
     </joint>
     <link name="body_3">
         <visual>
-            <origin xyz="0.0 0.0 0.0" rpy="0.0 0.0 0.0"/>
-            <geometry>
-                <mesh filename="package://lobster/meshes/body/LowerCover-Part3.stl" scale="${scale}"/>
-            </geometry>
-            <material name="red"/>
-        </visual>
+            <origin xyz="0.0 0.0 0.0" rpy="0.0 0.0 0.0" />
+            <geometry>
+                <mesh filename="package://lobster/meshes/body/LowerCover-Part3.stl" scale="${scale}" />
+            </geometry>
+            <material name="red" />
+        </visual>
+        <collision>
+            <origin xyz="0.0 0.0 0.0" rpy="0.0 0.0 0.0" />
+            <geometry>
+                <mesh filename="package://lobster/meshes/body/LowerCover-Part3.stl" scale="${scale}" />
+            </geometry>
+        </collision>
+        <xacro:default_inertial mass="1" />
     </link>
     <joint name="lower_body_3" type="fixed">
-        <parent link="base_link"/>
-        <child link="body_3"/>
-        <origin xyz="-0.043 0.046 0" rpy="0.0 0.0 ${PI/2}"/>
+        <parent link="base_link" />
+        <child link="body_3" />
+        <origin xyz="-0.043 0.046 0" rpy="0.0 0.0 ${PI/2}" />
     </joint>
     <link name="body_4">
         <visual>
-            <origin xyz="0.0 0.0 0.0" rpy="0.0 0.0 0.0"/>
-            <geometry>
-                <mesh filename="package://lobster/meshes/body/LowerCover-Part4.stl" scale="${scale}"/>
-            </geometry>
-            <material name="red"/>
-        </visual>
+            <origin xyz="0.0 0.0 0.0" rpy="0.0 0.0 0.0" />
+            <geometry>
+                <mesh filename="package://lobster/meshes/body/LowerCover-Part4.stl" scale="${scale}" />
+            </geometry>
+            <material name="red" />
+        </visual>
+        <collision>
+            <origin xyz="0.0 0.0 0.0" rpy="0.0 0.0 0.0" />
+            <geometry>
+                <mesh filename="package://lobster/meshes/body/LowerCover-Part4.stl" scale="${scale}" />
+            </geometry>
+        </collision>
+        <xacro:default_inertial mass="1" />
     </link>
     <joint name="lower_body_4" type="fixed">
-        <parent link="base_link"/>
-        <child link="body_4"/>
-        <origin xyz="-0.043 0.046 0" rpy="0.0 0.0 ${PI/2}"/> <!-- -0.043 0.046 0 -->
+        <parent link="base_link" />
+        <child link="body_4" />
+        <origin xyz="-0.043 0.046 0" rpy="0.0 0.0 ${PI/2}" /> <!-- -0.043 0.046 0 -->
     </joint>
     <link name="body_5">
@@ -68,4 +96,13 @@
             <material name="black" />
         </visual>
+        <collision>
+            <origin xyz="0.0 0.0 0.0" rpy="0.0 0.0 ${PI}" />
+            <geometry>
+                <mesh
+                    filename="package://lobster/meshes/body/UpperCover-Face-Part1.stl"
+                    scale="${scale}" />
+            </geometry>
+        </collision>
+        <xacro:default_inertial mass="1" />
     </link>
     <joint name="lower_body_5"
@@ -77,42 +114,67 @@
     <link name="body_6">
         <visual>
-            <origin xyz="0.0 0.0 0.0" rpy="0.0 0.0 0.0"/>
-            <geometry>
-                <mesh filename="package://lobster/meshes/body/UpperCover-Part2.stl" scale="${scale}"/>
-            </geometry>
-            <material name="red"/>
-        </visual>
+            <origin xyz="0.0 0.0 0.0" rpy="0.0 0.0 0.0" />
+            <geometry>
+                <mesh filename="package://lobster/meshes/body/UpperCover-Part2.stl" scale="${scale}" />
+            </geometry>
+            <material name="red" />
+        </visual>
+        <collision>
+            <origin xyz="0.0 0.0 0.0" rpy="0.0 0.0 0.0" />
+            <geometry>
+                <mesh filename="package://lobster/meshes/body/UpperCover-Part2.stl" scale="${scale}" />
+            </geometry>
+        </collision>
+        <xacro:default_inertial mass="1" />
     </link>
     <joint name="lower_body_6" type="fixed">
-        <parent link="base_link"/>
-        <child link="body_6"/>
+        <parent link="base_link" />
+        <child link="body_6" />
         <origin xyz="0.04 0 0.16" rpy="0.0 0.0 ${PI}" />
     </joint>
     <link name="body_7">
         <visual>
-            <origin xyz="0.0 0.0 0.0" rpy="0.0 0.0 0.0"/>
-            <geometry>
-                <mesh filename="package://lobster/meshes/body/Upper_Cover-With_Servo-Part3.stl" scale="${scale}"/>
-            </geometry>
-            <material name="red"/>
-        </visual>
+            <origin xyz="0.0 0.0 0.0" rpy="0.0 0.0 0.0" />
+            <geometry>
+                <mesh filename="package://lobster/meshes/body/Upper_Cover-With_Servo-Part3.stl"
+                    scale="${scale}" />
+            </geometry>
+            <material name="red" />
+        </visual>
+        <collision>
+            <origin xyz="0.0 0.0 0.0" rpy="0.0 0.0 0.0" />
+            <geometry>
+                <mesh filename="package://lobster/meshes/body/Upper_Cover-With_Servo-Part3.stl"
+                    scale="${scale}" />
+            </geometry>
+        </collision>
+        <xacro:default_inertial mass="1" />
     </link>
     <joint name="lower_body_7" type="fixed">
-        <parent link="base_link"/>
-        <child link="body_7"/>
+        <parent link="base_link" />
+        <child link="body_7" />
         <origin xyz="0.04 0 0.16" rpy="0.0 0.0 ${PI}" />
     </joint>
     <link name="body_8">
         <visual>
-            <origin xyz="0.0 0.0 0.0" rpy="0.0 0.0 0.0"/>
-            <geometry>
-                <mesh filename="package://lobster/meshes/body/Upper_Cover-With_Servo-Part4.stl" scale="${scale}"/>
-            </geometry>
-            <material name="red"/>
-        </visual>
+            <origin xyz="0.0 0.0 0.0" rpy="0.0 0.0 0.0" />
+            <geometry>
+                <mesh filename="package://lobster/meshes/body/Upper_Cover-With_Servo-Part4.stl"
+                    scale="${scale}" />
+            </geometry>
+            <material name="red" />
+        </visual>
+        <collision>
+            <origin xyz="0.0 0.0 0.0" rpy="0.0 0.0 0.0" />
+            <geometry>
+                <mesh filename="package://lobster/meshes/body/Upper_Cover-With_Servo-Part4.stl"
+                    scale="${scale}" />
+            </geometry>
+        </collision>
+        <xacro:default_inertial mass="1" />
     </link>
     <joint name="lower_body_8" type="fixed">
-        <parent link="base_link"/>
-        <child link="body_8"/>
+        <parent link="base_link" />
+        <child link="body_8" />
         <origin xyz="0.04 0 0.16" rpy="0.0 0.0 ${PI}" />
     </joint>
@@ -127,4 +189,13 @@
             <material name="red" />
         </visual>
+        <collision>
+            <origin xyz="0.0 0.0 0.0" rpy="0.0 ${PI} 0.0" />
+            <geometry>
+                <mesh
+                    filename="package://lobster/meshes/body/LidarTopPlate.stl"
+                    scale="${scale}" />
+            </geometry>
+        </collision>
+        <xacro:default_inertial mass="1" />
     </link>
     <joint name="lower_body_top"

File: lobster/urdf/lobster_chassi.xacro (robot description, xacro)
@@ -11,4 +11,11 @@
             <material name="blue"/>
         </visual>
+        <collision>
+            <origin xyz="0.0 0.0 0.0" rpy="0.0 0.0 ${-PI/2}"/>
+            <geometry>
+                <mesh filename="package://lobster/meshes/body/BasePlateHorizontal.stl" scale="${scale}"/>
+            </geometry>
+        </collision>
+        <xacro:default_inertial mass="1"/>
     </link>
     <joint name="virtual_joint" type="fixed">
@@ -24,4 +31,11 @@
             </geometry>
         </visual>
+        <collision>
+            <origin xyz="0.0 0.0 0.0" rpy="0.0 0.0 0.0"/>
+            <geometry>
+                <mesh filename="package://lobster/meshes/body/wheel.dae" scale="0.5 0.5 0.5"/>
+            </geometry>
+        </collision>
+        <xacro:default_inertial mass="1"/>
     </link>
     <joint name="left_wheel_joint" type="continuous">
@@ -38,4 +52,11 @@
             </geometry>
         </visual>
+        <collision>
+            <origin xyz="0.0 0.0 0.0" rpy="0.0 0.0 ${PI}"/>
+            <geometry>
+                <mesh filename="package://lobster/meshes/body/wheel.dae" scale="0.5 0.5 0.5"/>
+            </geometry>
+        </collision>
+        <xacro:default_inertial mass="1"/>
     </link>
     <joint name="joint_1" type="continuous">
@@ -52,4 +73,11 @@
             </geometry>
         </visual>
+        <collision>
+            <origin xyz="0.0 0.0 0.0" rpy="0.0 0.0 0.0"/>
+            <geometry>
+                <mesh filename="package://lobster/meshes/body/wheel.dae" scale="0.5 0.5 0.5"/>
+            </geometry>
+        </collision>
+        <xacro:default_inertial mass="1"/>
     </link>
     <joint name="joint_2" type="continuous">
@@ -66,4 +94,11 @@
             </geometry>
         </visual>
+        <collision>
+            <origin xyz="0.0 0.0 0.0" rpy="0.0 0.0 0.0"/>
+            <geometry>
+                <sphere radius="0.02"/>
+            </geometry>
+        </collision>
+        <xacro:default_inertial mass="1"/>
     </link>
     <joint name="caster_wheel_front" type="fixed">
@@ -79,4 +114,11 @@
             </geometry>
         </visual>
+        <collision>
+            <origin xyz="0.0 0.0 0.0" rpy="0.0 0.0 0.0"/>
+            <geometry>
+                <sphere radius="0.02"/>
+            </geometry>
+        </collision>
+        <xacro:default_inertial mass="1"/>
     </link>
     <joint name="caster_wheel_rear" type="fixed">

File: lobster/urdf/material.xacro (robot description, xacro)
@@ -22,4 +22,15 @@
         <color rgba="1 1 0 1"/>
     </material>
+    <xacro:property name="PI" value="3.14159" />
+    <xacro:property name="effort" value="30.0" />
+    <xacro:property name="velocity" value="10.0" />
+    <xacro:macro name="default_inertial" params="mass"> <!-- <xacro:default_inertial mass="1"/> -->
+        <inertial>
+            <mass value="${mass}" />
+            <inertia ixx="1.0" ixy="0.0" ixz="0.0"
+                     iyy="1.0" iyz="0.0"
+                     izz="1.0" />
+        </inertial>
+    </xacro:macro>
     <xacro:macro name="box_inertia" params="m l w h xyz rpy">
         <inertial>
